File: board/RISKYMSXCart.kicad_sch (KiCad schematic)
At the start: 35 parts, among them CN1 MSX_CART, IC8 LM1117MPX-3.3, J1 Conn_01x02, J2 Conn_01x02, J5 Conn_01x02, J7 USB_1, J8 Conn_01x02, SW1 SW_Push, U1 CH32V307VCT6

Commit message: Rev2 PCB
Parts:
- removed C7: 22uF, tfcart:PANASONIC_B, symbol tfcart-eagle-import:CPOL-USB
- removed J5: Conn_01x02, Connector_PinHeader_2.54mm:PinHeader_1x02_P2.54mm_Vertical, symbol Connector_Generic:Conn_01x02
- added C12, C14: C, Capacitor_SMD:C_0603_1608Metric_Pad1.08x0.95mm_HandSolder, symbol Device:C
- added C15, C16: C, Capacitor_SMD:C_0805_2012Metric_Pad1.18x1.45mm_HandSolder, symbol Device:C
- added C7: C, Capacitor_SMD:C_1206_3216Metric_Pad1.33x1.80mm_HandSolder, symbol Device:C
- added JP1: Jumper_2_Open, Jumper:SolderJumper-2_P1.3mm_Open_RoundedPad1.0x1.5mm, symbol Jumper:Jumper_2_Open
- added R9: R, Resistor_SMD:R_0603_1608Metric_Pad0.98x0.95mm_HandSolder, symbol Device:R
- added U2: MCP6001-OT, Package_TO_SOT_SMD:SOT-23-5, symbol Amplifier_Operational:MCP6001-OT
- added Y1: Crystal, Crystal:Crystal_SMD_5032-2Pin_5.0x3.2mm_HandSoldering, symbol Device:Crystal
- R2: value 10k -> R
Connections:
- net +5V: now also C7.1, U2.5 (V+)
- net GND: now also U1.37 (PB2/BOOT1(FT)), C15.1, C16.1, C7.2, R9.1, U2.2 (V-); no longer R2.1
- net SCC_AUD: now also C12.2; no longer U1.29 (PA4/ADC4/DAC0)
- net at U1.12 (OSC_IN): now also C15.2, Y1.2
- net at U1.13 (OSC_OUT): now also C16.2, Y1.1
- net BOOT1: no longer names the net of R2.2
- net BOOT1: now also R9.2, U2.4 (-); no longer U1.37 (PB2/BOOT1(FT))
- new net: C12.1, JP1.2 (B), R2.1, U2.1
- new net: C14.2, U2.3 (+)
- new net SCC_OUT: C14.1, JP1.1 (A), U1.29 (PA4/ADC4/DAC0)
- no-connect marks 36 -> 34

Commit message: Initial version 2.1
Parts:
- removed C15, C16: C, Capacitor_SMD:C_0805_2012Metric_Pad1.18x1.45mm_HandSolder, symbol Device:C
- removed D2, D3, D4: LED, LED_SMD:LED_0805_2012Metric_Pad1.15x1.40mm_HandSolder, symbol Device:LED
- removed JP1: Jumper_2_Open, Jumper:SolderJumper-2_P1.3mm_Open_RoundedPad1.0x1.5mm, symbol Jumper:Jumper_2_Open
- removed R6, R7, R8: 2.2k, Resistor_SMD:R_0603_1608Metric_Pad0.98x0.95mm_HandSolder, symbol Device:R
- removed SW1: SW_Push, Button_Switch_SMD:SW_SPST_Omron_B3FS-105xP, symbol Switch:SW_Push
- removed Y1: Crystal, Crystal:Crystal_SMD_5032-2Pin_5.0x3.2mm_HandSoldering, symbol Device:Crystal
- added C17, C18, C19, C20: C, Capacitor_SMD:C_0603_1608Metric_Pad1.08x0.95mm_HandSolder, symbol Device:C
- added R10: R, Resistor_SMD:R_0603_1608Metric_Pad0.98x0.95mm_HandSolder, symbol Device:R
Connections:
- net +5V: now also C18.2, C19.2
- net GND: now also C14.2, C18.1, C19.1
- net SCC_OUT: now also C20.1; no longer C14.1
- net at C12.1, R2.1, U2.1: now also C17.2
- net at U2.3 (+): now also C14.1, R10.2; no longer C14.2
- net at R2.2, R9.2, U2.4 (-): now also C17.1
- net BTN1 renamed LEDFLASH
- net LEDFLASH: now also D1.1 (K)
- net LED1: no longer names the net of U1.23 (PA0/WKUP/ADC0)
- net LED1: no longer D1.1 (K)
- net LED2: no longer names the net of U1.24 (PA1/ADC1)
- net LED3: no longer names the net of U1.25 (PA2/ADC2)
- net LED4: no longer names the net of U1.26 (PA3/ADC3)
- new net: C20.2, R10.1
- no-connect marks 34 -> 40
Other:
- moved on the sheet: C14

Commit message: schematic: add confirmed values for components with missing values
Signed-off-by: Albert Herranz <albert_herranz@yahoo.es>
Parts:
- C10, C11, C19, C2, C4, C5, C6, C7, C8: value C -> 100nF
- C12, C20: value C -> 4.7uF
- C14, C17: value C -> 1nF
- C18: value C -> 1uF
- C9: value 0.1μF -> 100nF
- F2: value Fuse -> 0.5A
- R1: value 10k -> 10K
- R10, R2, R4, R9: value R -> 10K
- R3: value 10k -> 220
- R5: value 2.2k -> 220
Changed lines of the file:
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@@
 			)
 		)
-		(property "Value" "2.2k"
+		(property "Value" "220"
 			(at 69.85 170.18 90)
 			(effects
@@
 			)
 		)
-		(property "Value" "C"
+		(property "Value" "100nF"
 			(at 31.75 76.1999 0)
 			(effects
@@
 			)
 		)
-		(property "Value" "R"
+		(property "Value" "10K"
 			(at 31.75 29.21 90)
 			(effects
@@
 			)
 		)
-		(property "Value" "R"
+		(property "Value" "10K"
 			(at 228.6 78.74 90)
 			(effects
@@
 			)
 		)
-		(property "Value" "C"
+		(property "Value" "4.7uF"
 			(at 269.24 80.01 90)
 			(effects
@@
 			)
 		)
-		(property "Value" "C"
+		(property "Value" "100nF"
 			(at 64.77 59.69 0)
 			(effects
@@
 			)
 		)
-		(property "Value" "C"
+		(property "Value" "1nF"
 			(at 243.84 99.06 90)
 			(effects
@@
 			)
 		)
-		(property "Value" "C"
+		(property "Value" "1nF"
 			(at 236.22 80.0099 0)
 			(effects
@@
 			)
 		)
-		(property "Value" "C"
+		(property "Value" "100nF"
 			(at 57.15 59.69 0)
 			(effects
@@
 			)
 		)
-		(property "Value" "10k"
+		(property "Value" "220"
 			(at 267.208 27.94 0)
 			(effects
@@
 			)
 		)
-		(property "Value" "R"
+		(property "Value" "10K"
 			(at 245.618 105.156 90)
 			(effects
@@
 			)
 		)
-		(property "Value" "C"
+		(property "Value" "100nF"
 			(at 34.29 59.69 0)
 			(effects
@@
 			)
 		)
-		(property "Value" "C"
+		(property "Value" "4.7uF"
 			(at 217.17 77.47 90)
 			(effects
@@
 			)
 		)
-		(property "Value" "10k"
+		(property "Value" "10K"
 			(at 55.372 36.576 90)
 			(effects
@@
 			)
 		)
-		(property "Value" "C"
+		(property "Value" "100nF"
 			(at 72.39 59.69 0)
 			(effects
@@
 			)
 		)
-		(property "Value" "C"
+		(property "Value" "100nF"
 			(at 80.01 59.69 0)
 			(effects
@@
 			)
 		)
-		(property "Value" "Fuse"
+		(property "Value" "0.5A"
 			(at 66.04 224.79 0)
 			(effects
@@
 			)
 		)
-		(property "Value" "C"
+		(property "Value" "1uF"
 			(at 247.65 72.3899 0)
 			(effects
@@
 			)
 		)
-		(property "Value" "0.1μF"
+		(property "Value" "100nF"
 			(at 38.1 38.1 0)
 			(effects
@@
 			)
 		)
-		(property "Value" "R"
+		(property "Value" "10K"
 			(at 233.68 105.664 90)
 			(effects
@@
 			)
 		)
-		(property "Value" "C"
+		(property "Value" "100nF"
 			(at 254 72.3899 0)
 			(effects
@@
 			)
 		)
-		(property "Value" "C"
+		(property "Value" "100nF"
 			(at 43.18 59.69 0)
 			(effects
@@
 			)
 		)
-		(property "Value" "C"
+		(property "Value" "100nF"
 			(at 48.26 59.69 0)
 			(effects
