File: board/RISKYMSXCart.kicad_pcb (KiCad board)
At the start: 4 copper layers, 71.9 x 55.5 mm, 38 parts, among them CN1 MSX_CART, IC8 LM1117MPX-3.3, J1 Conn_01x02, J2 Conn_01x02, J7 USB_1, J8 Conn_01x02, U1 CH32V307VCT6, U2 MCP6001-OT

Commit message: New PCB v2.2
Parts:
- removed @HOLE1 (x2): , 
- removed F2: 0.5A, Fuse:Fuse_1206_3216Metric_Pad1.42x1.75mm_HandSolder
- added G***: LOGO, footprints:RIKSYLOGOMINI, F.Cu at (123.8, 105.2)
- added R1: 150k, Resistor_SMD:R_0603_1608Metric_Pad0.98x0.95mm_HandSolder, B.Cu at (169.0, 85.8)
- added R3: 10k, Resistor_SMD:R_0603_1608Metric_Pad0.98x0.95mm_HandSolder, B.Cu at (160.5, 88.5)
- added U1: CH217K, Package_TO_SOT_SMD:SOT-23-6, B.Cu at (165.1, 86.0)
- C1: renamed from C7; value 100nF -> 100n
- C10: renamed from C1; value 100nF -> 100n
- C11: renamed from C3; value 10uF -> 10u
- C12: renamed from C20; value 4.7uF -> 4.7u
- C13: renamed from C14; value 1nF -> 1n
- C14: renamed from C18; value 1uF -> 1u
- C15: renamed from C17; value 1nF -> 1n
- C16: renamed from C13; value 1uF -> 1u
- C17: renamed from C19; value 100nF -> 100n
- C18: renamed from C12; value 4.7uF -> 4.7u
- C2: renamed from C10; value 100nF -> 100n
- C3: renamed from C9; value 100nF -> 100n
- C4: renamed from C11; value 100nF -> 100n
- C5: renamed from C2; value 100nF -> 100n
- C6: renamed from C4; value 100nF -> 100n
- C7: renamed from C5; value 100nF -> 100n
- C8: renamed from C6; value 100nF -> 100n
- C9: renamed from C8; value 100nF -> 100n
- U2: renamed from U1; value CH32V307VCT6 -> CH32V303VCT6
- moved C11 5.11 mm to (172.0, 88.1), turned to -90 degrees
- renumbered D5 to D2, IC8 to IC1, J8 to J1, J1 to J3, J7 to J4, R4 to R2, R1 to R4, R10 to R6, R9 to R7, R2 to R8, R3 to R9, U2 to U3
Connections:
- U2 pad 51: unconnected-(U1-PB12(FT)-Pad51) -> /VBUS
- U2 pad 52: unconnected-(U1-PB13(FT)-Pad52) -> /FLAG
Routing:
- net /VBUS: track 0.00 -> 21.9 mm, vias 0 -> 3
- net /FLAG: track 0.00 -> 16.6 mm, vias 0 -> 1
- net Net-(U1-ISET): track 0.00 -> 1.92 mm
- net GND: track 36.3 -> 37.9 mm, vias 27 -> 29
- net Net-(J4-VBUS): track 14.1 -> 15.6 mm
- net +5V: track 56.0 -> 55.2 mm
- net +3.3V: vias 15 -> 16
Other:
- board text added: "Rev.2.2"
- board text removed: "Rev.2.1"

Commit message: Update active layer and visible layers in RISKYMSXCart.kicad_prl configuration
Parts:
- moved C11 0.35 mm to (172.0, 87.8)
Routing:
- net +3.3V: track 38.0 -> 48.6 mm, vias 16 -> 15
- net GND: track 37.9 -> 46.3 mm, vias 29 -> 56
- net (no net): vias 0 -> 1
- added copper zone on B.Cu, net GND
- added copper zone on F.Cu, net GND
Other:
- board text removed: "SW"
